Commit message: ORB-SLAM working for cognifly

File: sim/cognifly/simple_quad.urdf (robot description, URDF)
Before this commit: robot simple_quad, 5 links, 4 joints
Joints:
- joint simple_quad_camera_joint: origin xyz=0.215 0 0.0 rpy=0 0 0 -> xyz=0.215 0 0.0 rpy=0 ${pi/2} 0

Commit message: First draft of map merging

File: sim/cognifly/simple_quad.urdf (robot description, URDF)
Before this commit: robot simple_quad, 5 links, 4 joints
Joints:
- joint simple_quad_camera_joint: origin xyz=0.215 0 0.0 rpy=0 ${pi/2} 0 -> xyz=0.215 0 0.0 rpy=0 ${pi/4} 0

Commit message: Revert "ORB-SLAM working for cognifly"

File: sim/cognifly/simple_quad.urdf (robot description, URDF)
Before this commit: robot simple_quad, 5 links, 4 joints
Joints:
- joint simple_quad_camera_joint: origin xyz=0.215 0 0.0 rpy=0 ${pi/2} 0 -> xyz=0.215 0 0.0 rpy=0 0 0
